File: PCB_OSCILLATOR/PCB_OSCILLATOR.kicad_pcb (KiCad board)
At the start: 2 copper layers, 94.4 x 37.1 mm, 102 parts, among them J1 Jumper, J10 Jumper, J11 Jumper, J12 Jumper, J13 Jumper, J14 Jumper, J15 Jumper, J16 Jumper, J2 Jumper, J3 Jumper, J4 Jumper, J5 Jumper, J6 Jumper, J7 Jumper, J8 Jumper, J9 Jumper, P1 CONN_01X04, P2 MCLK_EXTERNAL, P3 SPI_AD5270_1, P4 SPI_AD5270_2, P5 SPI_AD9833_1, P6 SPI_AD9833_2, P7 CONN_01X04, U1 AD5270, U10 ADR291, U2 AD8421, U3 AD9833, U4 AD5270, U5 AD8421, U6 AD9833, U7 ADG819, U8 ADP3334, U9 AD8651

Commit message: //
//
Parts:
- removed ? (x3): MountingHole_2.2mm_M2_Pad_Via, Mounting_Holes:MountingHole_2.2mm_M2_Pad_Via
Changed lines of the file:
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@@
-(kicad_pcb (version 4) (host pcbnew 4.0.2-stable)
+(kicad_pcb (version 4) (host pcbnew 4.0.6)
   (general
     (links 194)
     (no_connects 0)
-    (area 62.454999 65.874999 157.025001 103.145001)
+    (area 55.627143 65.155 163.922858 103.235)
     (thickness 1.6)
     (drawings 18)
     (tracks 776)
     (zones 0)
-    (modules 102)
+    (modules 99)
     (nets 61)
   )
@@
   )
   (setup
-    (last_trace_width 0.3)
+    (last_trace_width 0.2)
     (user_trace_width 0.3)
     (user_trace_width 0.35)
@@
     )
   )
-  (module Mounting_Holes:MountingHole_2.2mm_M2_Pad_Via (layer F.Cu)
-    (at 151.1 98.6)
-    (descr "Mounting Hole 2.2mm, M2")
-    (tags "mounting hole 2.2mm m2")
-    (fp_text reference "" (at 0 -3.2) (layer F.SilkS)
-      (effects (font (size 1 1) (thickness 0.15)))
-    )
-    (fp_text value MountingHole_2.2mm_M2_Pad_Via (at 0 3.2) (layer F.Fab)
-      (effects (font (size 1 1) (thickness 0.15)))
-    )
-    (fp_circle (center 0 0) (end 2.2 0) (layer Cmts.User) (width 0.15))
-    (fp_circle (center 0 0) (end 2.45 0) (layer F.CrtYd) (width 0.05))
-    (pad 1 thru_hole circle (at 0 0) (size 4.4 4.4) (drill 2.2) (layers *.Cu *.Mask F.SilkS))
-    (pad "" thru_hole circle (at 1.65 0) (size 0.6 0.6) (drill 0.4) (layers *.Cu *.Mask))
-    (pad "" thru_hole circle (at 1.166726 1.166726) (size 0.6 0.6) (drill 0.4) (layers *.Cu *.Mask))
-    (pad "" thru_hole circle (at 0 1.65) (size 0.6 0.6) (drill 0.4) (layers *.Cu *.Mask))
-    (pad "" thru_hole circle (at -1.166726 1.166726) (size 0.6 0.6) (drill 0.4) (layers *.Cu *.Mask))
-    (pad "" thru_hole circle (at -1.65 0) (size 0.6 0.6) (drill 0.4) (layers *.Cu *.Mask))
-    (pad "" thru_hole circle (at -1.166726 -1.166726) (size 0.6 0.6) (drill 0.4) (layers *.Cu *.Mask))
-    (pad "" thru_hole circle (at 0 -1.65) (size 0.6 0.6) (drill 0.4) (layers *.Cu *.Mask))
-    (pad "" thru_hole circle (at 1.166726 -1.166726) (size 0.6 0.6) (drill 0.4) (layers *.Cu *.Mask))
-  )
-  (module Mounting_Holes:MountingHole_2.2mm_M2_Pad_Via (layer F.Cu)
-    (at 68.45 96.17)
-    (descr "Mounting Hole 2.2mm, M2")
-    (tags "mounting hole 2.2mm m2")
-    (fp_text reference "" (at 0 -3.2) (layer F.SilkS)
-      (effects (font (size 1 1) (thickness 0.15)))
-    )
-    (fp_text value MountingHole_2.2mm_M2_Pad_Via (at 0 3.2) (layer F.Fab)
-      (effects (font (size 1 1) (thickness 0.15)))
-    )
-    (fp_circle (center 0 0) (end 2.2 0) (layer Cmts.User) (width 0.15))
-    (fp_circle (center 0 0) (end 2.45 0) (layer F.CrtYd) (width 0.05))
-    (pad 1 thru_hole circle (at 0 0) (size 4.4 4.4) (drill 2.2) (layers *.Cu *.Mask F.SilkS))
-    (pad "" thru_hole circle (at 1.65 0) (size 0.6 0.6) (drill 0.4) (layers *.Cu *.Mask))
-    (pad "" thru_hole circle (at 1.166726 1.166726) (size 0.6 0.6) (drill 0.4) (layers *.Cu *.Mask))
-    (pad "" thru_hole circle (at 0 1.65) (size 0.6 0.6) (drill 0.4) (layers *.Cu *.Mask))
-    (pad "" thru_hole circle (at -1.166726 1.166726) (size 0.6 0.6) (drill 0.4) (layers *.Cu *.Mask))
-    (pad "" thru_hole circle (at -1.65 0) (size 0.6 0.6) (drill 0.4) (layers *.Cu *.Mask))
-    (pad "" thru_hole circle (at -1.166726 -1.166726) (size 0.6 0.6) (drill 0.4) (layers *.Cu *.Mask))
-    (pad "" thru_hole circle (at 0 -1.65) (size 0.6 0.6) (drill 0.4) (layers *.Cu *.Mask))
-    (pad "" thru_hole circle (at 1.166726 -1.166726) (size 0.6 0.6) (drill 0.4) (layers *.Cu *.Mask))
-  )
-  (module Mounting_Holes:MountingHole_2.2mm_M2_Pad_Via (layer F.Cu)
-    (at 119.65 69.31)
-    (descr "Mounting Hole 2.2mm, M2")
-    (tags "mounting hole 2.2mm m2")
-    (fp_text reference "" (at 4.21 -1.25) (layer F.SilkS)
-      (effects (font (size 1 1) (thickness 0.15)))
-    )
-    (fp_text value MountingHole_2.2mm_M2_Pad_Via (at 0 3.2) (layer F.Fab)
-      (effects (font (size 1 1) (thickness 0.15)))
-    )
-    (fp_circle (center 0 0) (end 2.2 0) (layer Cmts.User) (width 0.15))
-    (fp_circle (center 0 0) (end 2.45 0) (layer F.CrtYd) (width 0.05))
-    (pad 1 thru_hole circle (at 0 0) (size 4.4 4.4) (drill 2.2) (layers *.Cu *.Mask F.SilkS))
-    (pad "" thru_hole circle (at 1.65 0) (size 0.6 0.6) (drill 0.4) (layers *.Cu *.Mask))
-    (pad "" thru_hole circle (at 1.166726 1.166726) (size 0.6 0.6) (drill 0.4) (layers *.Cu *.Mask))
-    (pad "" thru_hole circle (at 0 1.65) (size 0.6 0.6) (drill 0.4) (layers *.Cu *.Mask))
-    (pad "" thru_hole circle (at -1.166726 1.166726) (size 0.6 0.6) (drill 0.4) (layers *.Cu *.Mask))
-    (pad "" thru_hole circle (at -1.65 0) (size 0.6 0.6) (drill 0.4) (layers *.Cu *.Mask))
-    (pad "" thru_hole circle (at -1.166726 -1.166726) (size 0.6 0.6) (drill 0.4) (layers *.Cu *.Mask))
-    (pad "" thru_hole circle (at 0 -1.65) (size 0.6 0.6) (drill 0.4) (layers *.Cu *.Mask))
-    (pad "" thru_hole circle (at 1.166726 -1.166726) (size 0.6 0.6) (drill 0.4) (layers *.Cu *.Mask))
-  )
   (gr_text "SBS \nModule: 001" (at 140.17 98.82) (layer F.SilkS)
     (effects (font (size 1.5 1.5) (thickness 0.3)))
@@
       (pts
         (xy 122.32 87.54) (xy 119.36 90.56) (xy 115.72 90.56) (xy 115.76 85.36) (xy 115.76 85.28)
-        (xy 122.3 85.07) (xy 122.32 87.54)
+        (xy 122.3 85.07)
       )
     )
@@
         (xy 70.97 75.92) (xy 75.1 75.9) (xy 75.11 75.84) (xy 75.11 75.71) (xy 75.1 75.41)
         (xy 86.18 75.44) (xy 86.35 75.23) (xy 88.38 73.21) (xy 88.38 72.83) (xy 88.33 70.02)
-        (xy 84.73 70.08) (xy 84.69 66.18) (xy 125.79 66.19)
+        (xy 84.73 70.08) (xy 84.69 66.18)
       )
     )
@@
       (pts
         (xy 62.76 66.75) (xy 62.76 102.8) (xy 156.61 102.8) (xy 156.61 66.19) (xy 62.76 66.19)
-        (xy 62.76 66.75)
       )
     )
@@
         (xy 126.25 66.19) (xy 156.61 66.19) (xy 156.61 90.79) (xy 138.04 90.79) (xy 138.04 85.63)
         (xy 138.04 85.52) (xy 130.13 78.55) (xy 130.11 70.57) (xy 130.11 70.47) (xy 126.3 70.38)
-        (xy 126.25 66.19)
       )
     )
@@
     (polygon
       (pts
-        (xy 156.61 91.53) (xy 156.61 102.8) (xy 115.79 102.8) (xy 115.79 91.29) (xy 156.61 91.53)
+        (xy 156.61 91.53) (xy 156.61 102.8) (xy 115.79 102.8) (xy 115.79 91.29)
       )
     )
@@
         (xy 114.79 91.84) (xy 100.81 91.66) (xy 100.55 81.58) (xy 77.36 80.72) (xy 77.3 80.72)
         (xy 77.18 80.72) (xy 77.1 80.72) (xy 77.03 80.72) (xy 76.91 85.03) (xy 64.38 84.71)
-        (xy 64.21 84.71)
       )
     )
@@
       (pts
         (xy 84.8 70.6) (xy 87.85 70.59) (xy 87.83 72.81) (xy 85.94 74.7) (xy 80.94 74.78)
-        (xy 78.25 74.82) (xy 79.8 73.29) (xy 79.79 71.98) (xy 81.92 72.02) (xy 84.8 70.6)
+        (xy 78.25 74.82) (xy 79.8 73.29) (xy 79.79 71.98) (xy 81.92 72.02)
       )
     )
@@
         (xy 74.72 71.65) (xy 74.69 72.25) (xy 74.66 75.37) (xy 74.52 75.39) (xy 74.23 75.45)
         (xy 70.32 75.52) (xy 70.32 75.62) (xy 70.29 78.55) (xy 70.12 78.55) (xy 64.21 78.67)
-        (xy 64.21 71.57) (xy 74.72 71.65)
+        (xy 64.21 71.57)
       )
     )
@@
         (xy 84.23 69.66) (xy 84.22 70.13) (xy 82.01 71.35) (xy 79.67 71.35) (xy 79.2 71.37)
         (xy 79.23 73.18) (xy 77.75 74.7) (xy 75.21 74.8) (xy 75.22 71.23) (xy 62.76 71.14)
-        (xy 62.76 66.19) (xy 84.2 66.19) (xy 84.23 69.66)
+        (xy 62.76 66.19) (xy 84.2 66.19)
       )
     )
